File: Ananas-Core-avr-0.9.2/Ananas-core-0.9.2-no340G.sch (EAGLE design)
At the start: 56 parts, among them U1 MYSMD_ATMEGA168-20AU, Y1-16/20MHZ MYSMD2_RESONATORMU

Commit message: fix the endstop
Connections:
- removed net S1: J3.7, J5.3, U1.ADC6
- removed net S2: J3.6, J6.3, U1.ADC7
- net DA: now also J6.3
- net DL: now also J5.3
Changed lines of the file:
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@@
 <label x="2.54" y="83.82" size="1.778" layer="95"/>
+</segment>
+<segment>
+<pinref part="J5" gate="G$1" pin="3"/>
+<wire x1="-25.4" y1="137.16" x2="-20.32" y2="137.16" width="0.1524" layer="91"/>
+<label x="-20.32" y="137.16" size="1.778" layer="95"/>
 </segment>
 </net>
@@
 <wire x1="-2.54" y1="81.28" x2="2.54" y2="81.28" width="0.1524" layer="91"/>
 <label x="2.54" y="81.28" size="1.778" layer="95"/>
+</segment>
+<segment>
+<pinref part="J6" gate="G$1" pin="3"/>
+<wire x1="-25.4" y1="121.92" x2="-20.32" y2="121.92" width="0.1524" layer="91"/>
+<label x="-20.32" y="121.92" size="1.778" layer="95"/>
 </segment>
 </net>
@@
 </segment>
 </net>
-<net name="S1" class="0">
-<segment>
-<pinref part="U1" gate="G$1" pin="ADC6"/>
-<wire x1="-157.48" y1="127" x2="-162.56" y2="127" width="0.1524" layer="91"/>
-<label x="-167.64" y="127" size="1.778" layer="95"/>
-</segment>
-<segment>
-<pinref part="J3" gate="G$1" pin="7"/>
-<wire x1="-33.02" y1="78.74" x2="-30.48" y2="78.74" width="0.1524" layer="91"/>
-<label x="-30.48" y="78.74" size="1.778" layer="95"/>
-</segment>
-<segment>
-<pinref part="J5" gate="G$1" pin="3"/>
-<wire x1="-25.4" y1="137.16" x2="-20.32" y2="137.16" width="0.1524" layer="91"/>
-<label x="-22.86" y="137.16" size="1.778" layer="95"/>
-</segment>
-</net>
-<net name="S2" class="0">
-<segment>
-<pinref part="U1" gate="G$1" pin="ADC7"/>
-<wire x1="-157.48" y1="124.46" x2="-162.56" y2="124.46" width="0.1524" layer="91"/>
-<label x="-167.64" y="124.46" size="1.778" layer="95"/>
-</segment>
-<segment>
-<pinref part="J3" gate="G$1" pin="6"/>
-<wire x1="-33.02" y1="76.2" x2="-30.48" y2="76.2" width="0.1524" layer="91"/>
-<label x="-30.48" y="76.2" size="1.778" layer="95"/>
-</segment>
-<segment>
-<pinref part="J6" gate="G$1" pin="3"/>
-<wire x1="-25.4" y1="121.92" x2="-20.32" y2="121.92" width="0.1524" layer="91"/>
-<label x="-22.86" y="121.92" size="1.778" layer="95"/>
-</segment>
-</net>
